File: hardware/scanner.sch (EAGLE design)
At the start: 9 parts, among them K1 PIN20X2, U1 EEPROM24, U2 TPS61165DBV

Commit message: update hat
Parts:
- removed CFG: (no value), FLYFISH:PIN2_100
- added JP1, POWER: (no value), pinhead:PINHD-1X2
- SWITCH: device FLYFISH:PIN2_100 -> pinhead:PINHD-1X2
- U1: value EEPROM24 -> CAT24C32WI-GT3; device FLYFISH:EEPROM24 -> mbed-HDK-IC:CAT24C32WI-GT3
Connections:
- new net N$6: JP1.1, R3.2, U1.WP
- net +3V3: now also R3.1; no longer R3.2
- net GND: now also JP1.2, POWER.1, SWITCH.1, U1.VSS; no longer CFG.2, SWITCH.2, U1.GND
- net N$1: now also U1.SDA; no longer U1.SCL
- net N$2: now also POWER.2; no longer K1.27, R2.1, U1.SDA
- net N$3: now also K1.27, R2.1, U1.SCL; no longer CFG.1, R3.1, U1.WP
- net N$4: now also SWITCH.2; no longer SWITCH.1
Other:
- moved on the sheet: C1, R1, R2, R3, U2

Commit message: move eagle libs
Other:
- moved on the sheet: POWER
Changed lines of the file:
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@@
 <attribute name="VALUE" x="35.56" y="209.55" size="1.778" layer="96" rot="R270"/>
 </instance>
-<instance part="POWER" gate="G$1" x="38.1" y="53.34" smashed="yes" rot="R180">
-<attribute name="NAME" x="44.45" y="47.625" size="1.778" layer="95" rot="R180"/>
-<attribute name="VALUE" x="44.45" y="58.42" size="1.778" layer="96" rot="R180"/>
-</instance>
-<instance part="GND6" gate="1" x="48.26" y="45.72" smashed="yes">
-<attribute name="VALUE" x="45.72" y="43.18" size="1.778" layer="96"/>
-</instance>
-<instance part="P+3" gate="1" x="48.26" y="66.04" smashed="yes">
-<attribute name="VALUE" x="50.8" y="68.58" size="1.778" layer="96" rot="R180"/>
+<instance part="POWER" gate="G$1" x="203.2" y="142.24" smashed="yes" rot="R180">
+<attribute name="NAME" x="209.55" y="136.525" size="1.778" layer="95" rot="R180"/>
+<attribute name="VALUE" x="209.55" y="147.32" size="1.778" layer="96" rot="R180"/>
+</instance>
+<instance part="GND6" gate="1" x="213.36" y="134.62" smashed="yes">
+<attribute name="VALUE" x="210.82" y="132.08" size="1.778" layer="96"/>
+</instance>
+<instance part="P+3" gate="1" x="213.36" y="154.94" smashed="yes">
+<attribute name="VALUE" x="215.9" y="157.48" size="1.778" layer="96" rot="R180"/>
 </instance>
 </instances>
@@
 <segment>
 <pinref part="POWER" gate="G$1" pin="1"/>
-<wire x1="40.64" y1="50.8" x2="48.26" y2="50.8" width="0.1524" layer="91"/>
-<wire x1="48.26" y1="50.8" x2="48.26" y2="48.26" width="0.1524" layer="91"/>
+<wire x1="205.74" y1="139.7" x2="213.36" y2="139.7" width="0.1524" layer="91"/>
+<wire x1="213.36" y1="139.7" x2="213.36" y2="137.16" width="0.1524" layer="91"/>
 <pinref part="GND6" gate="1" pin="GND"/>
 </segment>
@@
 <segment>
 <pinref part="P+3" gate="1" pin="+5V"/>
-<wire x1="48.26" y1="63.5" x2="48.26" y2="60.96" width="0.1524" layer="91"/>
+<wire x1="213.36" y1="152.4" x2="213.36" y2="149.86" width="0.1524" layer="91"/>
 </segment>
 </net>
@@
 <segment>
 <pinref part="POWER" gate="G$1" pin="2"/>
-<wire x1="40.64" y1="53.34" x2="48.26" y2="53.34" width="0.1524" layer="91"/>
-<wire x1="48.26" y1="53.34" x2="48.26" y2="55.88" width="0.1524" layer="91"/>
-</segment>
-</net>
+<wire x1="205.74" y1="142.24" x2="213.36" y2="142.24" width="0.1524" layer="91"/>
+<wire x1="213.36" y1="142.24" x2="213.36" y2="144.78" width="0.1524" layer="91"/>
+</segment>
+</net>

Commit message: update pcb
Parts:
- added C2: 220nF, resistor:C-EUC0805K
- added C3: 4.7μF, resistor:C-EUC0805K
- added C4: 1μF, resistor:C-EUC0805K
- added D1: 40V 550mA, adafruit:DIODESOD-123
- added L1: 10 μH ±20% 1.49A, m-pad-2.1:D53LC
- added LED1, LED2: LW_W5SM-JYKY-JKQL-1, LW_W5SM-JYKY-JKQL-1:LW_W5SM-JYKY-JKQL-1
- added LED3, LED4, LED5: (no value), led:LEDCHIP-LED0805
- added R4: 0.57, resistor:R-EU_M0805
- added R5, R6, R7: 330, resistor:R-EU_M0805
Connections:
- new net N$10: C4.1, D1.C, LED1.A
- new net N$11: LED1.K, LED2.A
- new net N$13: LED3.A, R5.2
- new net N$16: K1.13, R6.1
- new net N$17: LED4.A, R6.2
- new net N$18: LED5.A, R7.2
- new net N$19: K1.11, R5.1
- new net N$20: K1.15, R7.1
- new net N$7: C2.1, U2.COMP
- new net N$8: LED2.K, R4.1, U2.FB
- new net N$9: D1.A, L1.2, U2.SW
- net +5V: now also C3.1, L1.1
- net GND: now also C2.2, C3.2, C4.2, LED3.C, LED4.C, LED5.C, R4.2
Other:
- moved on the sheet: C1, JP1, K1, POWER, R1, R2, R3, SWITCH, U1, U2

Commit message: update pcb
Parts:
- removed POWER: (no value), pinhead:PINHD-1X2
- added JP2: (no value), pinhead:PINHD-2X2
Connections:
- removed net N$2: POWER.2
- net +5V: now also JP2.1, JP2.2
- net GND: now also JP2.3, JP2.4; no longer POWER.1
Changed lines of the file:
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@@
 <part name="SWITCH" library="pinhead" library_urn="urn:adsk.eagle:library:325" deviceset="PINHD-1X2" device="" package3d_urn="urn:adsk.eagle:package:22435/2"/>
 <part name="JP1" library="pinhead" library_urn="urn:adsk.eagle:library:325" deviceset="PINHD-1X2" device="" package3d_urn="urn:adsk.eagle:package:22435/2"/>
-<part name="POWER" library="pinhead" library_urn="urn:adsk.eagle:library:325" deviceset="PINHD-1X2" device="" package3d_urn="urn:adsk.eagle:package:22435/2"/>
 <part name="GND6" library="supply1" deviceset="GND" device=""/>
 <part name="P+3" library="supply1" deviceset="+5V" device=""/>
@@
 <attribute name="TOLERANCE" value="5%"/>
 </part>
+<part name="JP2" library="pinhead" library_urn="urn:adsk.eagle:library:325" deviceset="PINHD-2X2" device="" package3d_urn="urn:adsk.eagle:package:22455/2"/>
 </parts>
 <sheets>
@@
 <attribute name="VALUE" x="68.58" y="209.55" size="1.778" layer="96" rot="R270"/>
 </instance>
-<instance part="POWER" gate="G$1" x="35.56" y="63.5" smashed="yes" rot="R180">
-<attribute name="NAME" x="41.91" y="57.785" size="1.778" layer="95" rot="R180"/>
-<attribute name="VALUE" x="41.91" y="68.58" size="1.778" layer="96" rot="R180"/>
-</instance>
-<instance part="GND6" gate="1" x="45.72" y="55.88" smashed="yes">
-<attribute name="VALUE" x="43.18" y="53.34" size="1.778" layer="96"/>
-</instance>
-<instance part="P+3" gate="1" x="45.72" y="76.2" smashed="yes">
-<attribute name="VALUE" x="48.26" y="78.74" size="1.778" layer="96" rot="R180"/>
+<instance part="GND6" gate="1" x="81.28" y="58.42" smashed="yes">
+<attribute name="VALUE" x="78.74" y="55.88" size="1.778" layer="96"/>
+</instance>
+<instance part="P+3" gate="1" x="81.28" y="78.74" smashed="yes">
+<attribute name="VALUE" x="83.82" y="81.28" size="1.778" layer="96" rot="R180"/>
 </instance>
 <instance part="C2" gate="G$1" x="160.02" y="154.94" smashed="yes">
@@
 <attribute name="NAME" x="50.5714" y="154.94" size="1.778" layer="95" rot="R90"/>
 <attribute name="VALUE" x="52.832" y="154.94" size="1.778" layer="96" rot="R90"/>
+</instance>
+<instance part="JP2" gate="A" x="71.12" y="63.5" smashed="yes">
+<attribute name="NAME" x="62.23" y="69.215" size="1.778" layer="95"/>
+<attribute name="VALUE" x="62.23" y="58.42" size="1.778" layer="96"/>
 </instance>
 </instances>
@@
 </segment>
 <segment>
-<pinref part="POWER" gate="G$1" pin="1"/>
-<wire x1="38.1" y1="60.96" x2="45.72" y2="60.96" width="0.1524" layer="91"/>
-<wire x1="45.72" y1="60.96" x2="45.72" y2="58.42" width="0.1524" layer="91"/>
+<wire x1="73.66" y1="63.5" x2="81.28" y2="63.5" width="0.1524" layer="91"/>
+<wire x1="81.28" y1="63.5" x2="81.28" y2="60.96" width="0.1524" layer="91"/>
 <pinref part="GND6" gate="1" pin="GND"/>
+<pinref part="JP2" gate="A" pin="4"/>
+<pinref part="JP2" gate="A" pin="3"/>
+<wire x1="66.04" y1="63.5" x2="73.66" y2="63.5" width="0.1524" layer="91"/>
+<junction x="73.66" y="63.5"/>
 </segment>
 <segment>
@@
 <segment>
 <pinref part="P+3" gate="1" pin="+5V"/>
-<wire x1="45.72" y1="73.66" x2="45.72" y2="71.12" width="0.1524" layer="91"/>
+<wire x1="73.66" y1="66.04" x2="81.28" y2="66.04" width="0.1524" layer="91"/>
+<pinref part="JP2" gate="A" pin="2"/>
+<wire x1="81.28" y1="66.04" x2="81.28" y2="76.2" width="0.1524" layer="91"/>
+<pinref part="JP2" gate="A" pin="1"/>
+<wire x1="66.04" y1="66.04" x2="73.66" y2="66.04" width="0.1524" layer="91"/>
+<junction x="73.66" y="66.04"/>
 </segment>
 </net>
@@
 </segment>
 </net>
-<net name="N$2" class="0">
-<segment>
-<pinref part="POWER" gate="G$1" pin="2"/>
-<wire x1="38.1" y1="63.5" x2="45.72" y2="63.5" width="0.1524" layer="91"/>
-<wire x1="45.72" y1="63.5" x2="45.72" y2="66.04" width="0.1524" layer="91"/>
-</segment>
-</net>

Commit message: added camera mounting holes
Parts:
- renumbered JP2 to POWER
Changed lines of the file:
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@@
 <attribute name="TOLERANCE" value="5%"/>
 </part>
-<part name="JP2" library="pinhead" library_urn="urn:adsk.eagle:library:325" deviceset="PINHD-2X2" device="" package3d_urn="urn:adsk.eagle:package:22455/2"/>
+<part name="POWER" library="pinhead" library_urn="urn:adsk.eagle:library:325" deviceset="PINHD-2X2" device="" package3d_urn="urn:adsk.eagle:package:22455/2"/>
 </parts>
 <sheets>
@@
 <attribute name="VALUE" x="68.58" y="209.55" size="1.778" layer="96" rot="R270"/>
 </instance>
-<instance part="GND6" gate="1" x="81.28" y="58.42" smashed="yes">
-<attribute name="VALUE" x="78.74" y="55.88" size="1.778" layer="96"/>
+<instance part="GND6" gate="1" x="81.28" y="53.34" smashed="yes">
+<attribute name="VALUE" x="78.74" y="50.8" size="1.778" layer="96"/>
 </instance>
 <instance part="P+3" gate="1" x="81.28" y="78.74" smashed="yes">
@@
 <attribute name="VALUE" x="52.832" y="154.94" size="1.778" layer="96" rot="R90"/>
 </instance>
-<instance part="JP2" gate="A" x="71.12" y="63.5" smashed="yes">
+<instance part="POWER" gate="A" x="71.12" y="63.5" smashed="yes">
 <attribute name="NAME" x="62.23" y="69.215" size="1.778" layer="95"/>
 <attribute name="VALUE" x="62.23" y="58.42" size="1.778" layer="96"/>
@@
 <segment>
 <wire x1="73.66" y1="63.5" x2="81.28" y2="63.5" width="0.1524" layer="91"/>
-<wire x1="81.28" y1="63.5" x2="81.28" y2="60.96" width="0.1524" layer="91"/>
+<wire x1="81.28" y1="63.5" x2="81.28" y2="55.88" width="0.1524" layer="91"/>
 <pinref part="GND6" gate="1" pin="GND"/>
-<pinref part="JP2" gate="A" pin="4"/>
-<pinref part="JP2" gate="A" pin="3"/>
+<pinref part="POWER" gate="A" pin="4"/>
+<pinref part="POWER" gate="A" pin="3"/>
 <wire x1="66.04" y1="63.5" x2="73.66" y2="63.5" width="0.1524" layer="91"/>
 <junction x="73.66" y="63.5"/>
@@
 <pinref part="P+3" gate="1" pin="+5V"/>
 <wire x1="73.66" y1="66.04" x2="81.28" y2="66.04" width="0.1524" layer="91"/>
-<pinref part="JP2" gate="A" pin="2"/>
+<pinref part="POWER" gate="A" pin="2"/>
 <wire x1="81.28" y1="66.04" x2="81.28" y2="76.2" width="0.1524" layer="91"/>
-<pinref part="JP2" gate="A" pin="1"/>
+<pinref part="POWER" gate="A" pin="1"/>
 <wire x1="66.04" y1="66.04" x2="73.66" y2="66.04" width="0.1524" layer="91"/>
 <junction x="73.66" y="66.04"/>

Commit message: new power connector
Parts:
- POWER: value (none) -> 2.1MMJACKTHM; device pinhead:PINHD-2X2 -> adafruit:2.1MMJACKTHM
Connections:
- net +5V: now also POWER.TIP; no longer POWER.1, POWER.2
- net GND: now also POWER.RING, POWER.RING_SW; no longer POWER.3, POWER.4
Changed lines of the file:
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@@
 <attribute name="TOLERANCE" value="5%"/>
 </part>
-<part name="POWER" library="pinhead" library_urn="urn:adsk.eagle:library:325" deviceset="PINHD-2X2" device="" package3d_urn="urn:adsk.eagle:package:22455/2"/>
+<part name="POWER" library="adafruit" library_urn="urn:adsk.eagle:library:420" deviceset="2.1MMJACK" device="THM" package3d_urn="urn:adsk.eagle:package:6240341/1"/>
 </parts>
 <sheets>
@@
 <attribute name="VALUE" x="52.832" y="154.94" size="1.778" layer="96" rot="R90"/>
 </instance>
-<instance part="POWER" gate="A" x="71.12" y="63.5" smashed="yes">
-<attribute name="NAME" x="62.23" y="69.215" size="1.778" layer="95"/>
-<attribute name="VALUE" x="62.23" y="58.42" size="1.778" layer="96"/>
+<instance part="POWER" gate="G$1" x="68.58" y="63.5" smashed="yes">
+<attribute name="NAME" x="66.04" y="68.58" size="1.27" layer="95"/>
 </instance>
 </instances>
@@
 </segment>
 <segment>
-<wire x1="73.66" y1="63.5" x2="81.28" y2="63.5" width="0.1524" layer="91"/>
-<wire x1="81.28" y1="63.5" x2="81.28" y2="55.88" width="0.1524" layer="91"/>
+<wire x1="81.28" y1="60.96" x2="81.28" y2="55.88" width="0.1524" layer="91"/>
 <pinref part="GND6" gate="1" pin="GND"/>
-<pinref part="POWER" gate="A" pin="4"/>
-<pinref part="POWER" gate="A" pin="3"/>
-<wire x1="66.04" y1="63.5" x2="73.66" y2="63.5" width="0.1524" layer="91"/>
-<junction x="73.66" y="63.5"/>
+<pinref part="POWER" gate="G$1" pin="RING_SW"/>
+<pinref part="POWER" gate="G$1" pin="RING"/>
+<wire x1="73.66" y1="63.5" x2="73.66" y2="60.96" width="0.1524" layer="91"/>
+<wire x1="73.66" y1="60.96" x2="81.28" y2="60.96" width="0.1524" layer="91"/>
+<junction x="73.66" y="60.96"/>
 </segment>
 <segment>
@@
 <pinref part="P+3" gate="1" pin="+5V"/>
 <wire x1="73.66" y1="66.04" x2="81.28" y2="66.04" width="0.1524" layer="91"/>
-<pinref part="POWER" gate="A" pin="2"/>
 <wire x1="81.28" y1="66.04" x2="81.28" y2="76.2" width="0.1524" layer="91"/>
-<pinref part="POWER" gate="A" pin="1"/>
-<wire x1="66.04" y1="66.04" x2="73.66" y2="66.04" width="0.1524" layer="91"/>
-<junction x="73.66" y="66.04"/>
+<pinref part="POWER" gate="G$1" pin="TIP"/>
 </segment>
 </net>

Commit message: rename routes
Parts:
- renumbered SWITCH to TRIGGER
Connections:
- net N$1 renamed EEPROM_SDA
- net N$16 renamed LED4
- net N$19 renamed LED3
- net N$20 renamed LED5
- net N$3 renamed EEPROM_SCL
- net N$4 renamed TRIGGER
- net N$6 renamed EEPROM_WP
Changed lines of the file:
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@@
 </part>
 <part name="+3V2" library="supply1" deviceset="+3V3" device=""/>
-<part name="SWITCH" library="pinhead" library_urn="urn:adsk.eagle:library:325" deviceset="PINHD-1X2" device="" package3d_urn="urn:adsk.eagle:package:22435/2"/>
+<part name="TRIGGER" library="pinhead" library_urn="urn:adsk.eagle:library:325" deviceset="PINHD-1X2" device="" package3d_urn="urn:adsk.eagle:package:22435/2"/>
 <part name="JP1" library="pinhead" library_urn="urn:adsk.eagle:library:325" deviceset="PINHD-1X2" device="" package3d_urn="urn:adsk.eagle:package:22435/2"/>
 <part name="GND6" library="supply1" deviceset="GND" device=""/>
@@
 <attribute name="VALUE" x="129.54" y="243.84" size="1.778" layer="96" rot="R180"/>
 </instance>
-<instance part="SWITCH" gate="G$1" x="71.12" y="96.52" smashed="yes" rot="R180">
+<instance part="TRIGGER" gate="G$1" x="71.12" y="96.52" smashed="yes" rot="R180">
 <attribute name="NAME" x="77.47" y="90.805" size="1.778" layer="95" rot="R180"/>
 <attribute name="VALUE" x="77.47" y="101.6" size="1.778" layer="96" rot="R180"/>
@@
 <pinref part="GND4" gate="1" pin="GND"/>
 <wire x1="81.28" y1="93.98" x2="81.28" y2="91.44" width="0.1524" layer="91"/>
-<pinref part="SWITCH" gate="G$1" pin="1"/>
+<pinref part="TRIGGER" gate="G$1" pin="1"/>
 </segment>
 <segment>
@@
 </segment>
 </net>
-<net name="N$1" class="0">
+<net name="EEPROM_SDA" class="0">
 <segment>
 <pinref part="R1" gate="G$1" pin="1"/>
@@
 </segment>
 </net>
-<net name="N$4" class="0">
+<net name="TRIGGER" class="0">
 <segment>
 <wire x1="73.66" y1="96.52" x2="106.68" y2="96.52" width="0.1524" layer="91"/>
@@
 <pinref part="K1" gate="G$1" pin="16"/>
 <wire x1="106.68" y1="157.48" x2="91.44" y2="157.48" width="0.1524" layer="91"/>
-<pinref part="SWITCH" gate="G$1" pin="2"/>
+<pinref part="TRIGGER" gate="G$1" pin="2"/>
 </segment>
 </net>
@@
 </segment>
 </net>
-<net name="N$6" class="0">
+<net name="EEPROM_WP" class="0">
 <segment>
 <pinref part="U1" gate="A" pin="WP"/>
@@
 </segment>
 </net>
-<net name="N$3" class="0">
+<net name="EEPROM_SCL" class="0">
 <segment>
 <pinref part="R2" gate="G$1" pin="1"/>
@@
 </segment>
 </net>
-<net name="N$16" class="0">
+<net name="LED4" class="0">
 <segment>
 <pinref part="K1" gate="G$1" pin="13"/>
@@
 </segment>
 </net>
-<net name="N$19" class="0">
+<net name="LED3" class="0">
 <segment>
 <pinref part="K1" gate="G$1" pin="11"/>
@@
 </segment>
 </net>
-<net name="N$20" class="0">
+<net name="LED5" class="0">
 <segment>
 <pinref part="K1" gate="G$1" pin="15"/>
