File: hardware/scanner.brd (EAGLE design)
At the start: 65 x 56 mm, 25 parts, among them K1 PIN20X2, U1 CAT24C32WI-GT3, U2 TPS61165DBV

Commit message: update board
Parts:
- removed R8: 10k, resistor:M0805
- renumbered K1 to GPIO
Connections:
- net N$5 renamed LED_PWM
- net N$8 renamed LED_FB
- net N$9 renamed LED_SW
- net +5V: no longer R8.2
- net GND: now also LED1.3, LED2.3
- net TRIGGER: no longer R8.1
Routing:
- net +3V3: track 63.3 -> 84.6 mm
- net +5V: track 82.6 -> 76.8 mm
- net TRIGGER: track 52.5 -> 46.8 mm
Changed lines of the file:
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@@
 <text x="32.635" y="28" size="1.778" layer="25" align="center">CAMERA
 MODULE</text>
-<text x="61" y="8" size="2.54" layer="25" rot="R90">Scanner HAT</text>
-<text x="62" y="8" size="0.8128" layer="25" rot="R90" align="center-left">shopper.ink ©    v1.0</text>
+<text x="61" y="8" size="2.1844" layer="25" font="fixed" rot="R90">Scanner HAT</text>
+<text x="62" y="8" size="1.016" layer="25" font="fixed" rot="R90" align="center-left">shopper.ink © v1.0</text>
 <circle x="3.5" y="52.5" radius="1.55" width="3.1" layer="42"/>
-<text x="8" y="23" size="0.8128" layer="25" rot="R180" align="center">GND</text>
-<text x="7.605" y="20.545" size="0.8128" layer="25" align="center">+5V</text>
-<text x="8" y="25.635" size="0.8128" layer="25" rot="R180" align="center">CTRL</text>
+<text x="8" y="23" size="0.8128" layer="25" font="fixed" rot="R180" align="center">GND</text>
+<text x="7.605" y="20.545" size="0.8128" layer="25" font="fixed" align="center">+5V</text>
+<text x="8" y="25.635" size="0.8128" layer="25" font="fixed" rot="R180" align="center">CTRL</text>
 </plain>
 <attributes>
@@
 <description language="zh">&lt;b&gt;Seeed Studio EAGLE Design Rules&lt;/b&gt;
 </description>
-<param name="layerSetup" value="(1*16)"/>
+<param name="layerSetup" value="(1+2*15+16)"/>
 <param name="mtCopper" value="0.035mm 0.035mm 0.035mm 0.035mm 0.035mm 0.035mm 0.035mm 0.035mm 0.035mm 0.035mm 0.035mm 0.035mm 0.035mm 0.035mm 0.035mm 0.035mm"/>
 <param name="mtIsolate" value="1.5mm 0.15mm 0.2mm 0.15mm 0.2mm 0.15mm 0.2mm 0.15mm 0.2mm 0.15mm 0.2mm 0.15mm 0.2mm 0.15mm 0.2mm"/>
@@
 </autorouter>
 <elements>
-<element name="K1" library="FLYFISH" package="PIN_20X2" value="PIN20X2" x="32.5" y="52.5" smashed="yes">
+<element name="GPIO" library="FLYFISH" package="PIN_20X2" value="PIN20X2" x="32.5" y="52.5" smashed="yes">
 <attribute name="VALUE" x="45.2" y="48.309" size="1.27" layer="27" ratio="10"/>
 </element>
@@
 <attribute name="MF" value="MOLEX" x="5" y="23" size="1.778" layer="27" rot="R270" display="off"/>
 <attribute name="MPN" value="" x="5" y="23" size="1.778" layer="27" rot="R270" display="off"/>
-<attribute name="NAME" x="1" y="23" size="1.016" layer="25" ratio="10" rot="R270" align="center"/>
+<attribute name="NAME" x="4" y="28" size="1.016" layer="25" font="fixed" ratio="10" align="center"/>
 <attribute name="OC_FARNELL" value="unknown" x="5" y="23" size="1.778" layer="27" rot="R270" display="off"/>
 <attribute name="OC_NEWARK" value="unknown" x="5" y="23" size="1.778" layer="27" rot="R270" display="off"/>
 <attribute name="VALUE" x="2.5601" y="18.3279" size="0.8128" layer="27" ratio="10" rot="R180"/>
 </element>
-<element name="R8" library="resistor" package="M0805" value="10k" x="10" y="23" smashed="yes" rot="R270">
-<attribute name="NAME" x="10.016" y="26.016" size="0.8128" layer="25" rot="R270" align="center-left"/>
-<attribute name="TOLERANCE" value="5%" x="10" y="23" size="1.778" layer="27" rot="R270" display="off"/>
-<attribute name="VALUE" x="7.714" y="24.016" size="1.27" layer="27" rot="R270"/>
-</element>
 </elements>
 <signals>
@@
 <signal name="GND">
 <contactref element="C1" pad="2"/>
-<contactref element="K1" pad="9"/>
-<contactref element="K1" pad="25"/>
-<contactref element="K1" pad="39"/>
-<contactref element="K1" pad="6"/>
-<contactref element="K1" pad="14"/>
-<contactref element="K1" pad="20"/>
-<contactref element="K1" pad="30"/>
-<contactref element="K1" pad="34"/>
+<contactref element="GPIO" pad="9"/>
+<contactref element="GPIO" pad="25"/>
+<contactref element="GPIO" pad="39"/>
+<contactref element="GPIO" pad="6"/>
+<contactref element="GPIO" pad="14"/>
+<contactref element="GPIO" pad="20"/>
+<contactref element="GPIO" pad="30"/>
+<contactref element="GPIO" pad="34"/>
 <contactref element="U1" pad="4"/>
 <contactref element="U1" pad="3"/>
@@
 <wire x1="19" y1="3.95" x2="19.05" y2="4" width="0.3048" layer="1"/>
 <contactref element="TRIGGER" pad="2"/>
+<contactref element="LED1" pad="3"/>
+<contactref element="LED2" pad="3"/>
 </signal>
 <signal name="+3V3">
@@
 <contactref element="R2" pad="2"/>
 <contactref element="R1" pad="2"/>
-<contactref element="K1" pad="1"/>
-<contactref element="K1" pad="17"/>
+<contactref element="GPIO" pad="1"/>
+<contactref element="GPIO" pad="17"/>
 <contactref element="U1" pad="8"/>
 <contactref element="R3" pad="1"/>
 <wire x1="62" y1="46.905" x2="61.4638" y2="46.905" width="0.1524" layer="1"/>
-<wire x1="28.69" y1="51.23" x2="28.69" y2="49.31" width="0.3048" layer="1"/>
-<wire x1="28.69" y1="49.31" x2="29" y2="49" width="0.3048" layer="1"/>
-<wire x1="29" y1="49" x2="62" y2="49" width="0.3048" layer="1"/>
+<wire x1="28.69" y1="51.23" x2="28.69" y2="50.31" width="0.3048" layer="1"/>
+<wire x1="28.69" y1="50.31" x2="29" y2="50" width="0.3048" layer="1"/>
+<wire x1="29" y1="50" x2="62" y2="50" width="0.3048" layer="1"/>
 <wire x1="61.05" y1="38" x2="61" y2="38.05" width="0.3048" layer="1"/>
-<wire x1="62" y1="49" x2="63" y2="48" width="0.3048" layer="1"/>
-<wire x1="63" y1="48" x2="63" y2="47" width="0.3048" layer="1"/>
+<wire x1="62" y1="50" x2="63" y2="49" width="0.3048" layer="1"/>
+<wire x1="63" y1="49" x2="63" y2="47" width="0.3048" layer="1"/>
 <wire x1="63" y1="47" x2="63" y2="38" width="0.3048" layer="1"/>
 <wire x1="63" y1="38" x2="63" y2="33" width="0.3048" layer="1"/>
@@
 <wire x1="57" y1="38.05" x2="59" y2="38.05" width="0.3048" layer="1"/>
 <wire x1="59" y1="38.05" x2="61" y2="38.05" width="0.3048" layer="1"/>
-<wire x1="8.37" y1="51.23" x2="28.69" y2="51.23" width="0" layer="19" extent="1-1"/>
+<wire x1="28.69" y1="50.31" x2="28.38" y2="50" width="0.3048" layer="1"/>
+<wire x1="9" y1="50" x2="8.37" y2="50.63" width="0.3048" layer="1"/>
+<wire x1="8.37" y1="50.63" x2="8.37" y2="51.23" width="0.3048" layer="1"/>
+<wire x1="28.38" y1="50" x2="9" y2="50" width="0.3048" layer="1"/>
 </signal>
 <signal name="EEPROM_SDA">
 <contactref element="R1" pad="1"/>
-<contactref element="K1" pad="28"/>
+<contactref element="GPIO" pad="28"/>
 <contactref element="U1" pad="5"/>
 <wire x1="59" y1="49" x2="43" y2="49" width="0.2032" layer="16"/>
@@
 </signal>
 <signal name="+5V">
-<contactref element="K1" pad="2"/>
-<contactref element="K1" pad="4"/>
+<contactref element="GPIO" pad="2"/>
+<contactref element="GPIO" pad="4"/>
 <contactref element="U2" pad="1"/>
 <wire x1="8.37" y1="53.77" x2="10.91" y2="53.77" width="0.8128" layer="1"/>
@@
 <wire x1="4" y1="9" x2="2" y2="11" width="0.8128" layer="1"/>
 <contactref element="TRIGGER" pad="1"/>
-<wire x1="2" y1="11" x2="2" y2="21" width="0.8128" layer="1"/>
-<wire x1="2" y1="21" x2="2" y2="46" width="0.8128" layer="1"/>
-<wire x1="5" y1="20.46" x2="4.46" y2="21" width="0.508" layer="1"/>
-<wire x1="4.46" y1="21" x2="2" y2="21" width="0.508" layer="1"/>
-<contactref element="R8" pad="2"/>
-<wire x1="9.41" y1="21.46" x2="6" y2="21.46" width="0.508" layer="1"/>
-<wire x1="5" y1="20.46" x2="6" y2="21.46" width="0.508" layer="1"/>
-<wire x1="9.41" y1="21.46" x2="10" y2="22.05" width="0.508" layer="1"/>
+<wire x1="2" y1="11" x2="2" y2="20.32" width="0.8128" layer="1"/>
+<wire x1="2" y1="20.32" x2="2" y2="46" width="0.8128" layer="1"/>
+<wire x1="5" y1="20.46" x2="2.14" y2="20.46" width="0.508" layer="1"/>
+<wire x1="2.14" y1="20.46" x2="2" y2="20.32" width="0.508" layer="1"/>
 </signal>
 <signal name="TRIGGER">
-<contactref element="K1" pad="16"/>
+<contactref element="GPIO" pad="16"/>
 <wire x1="8" y1="48" x2="9" y2="49" width="0.2032" layer="16"/>
 <wire x1="9" y1="49" x2="18.365" y2="49" width="0.2032" layer="16"/>
@@
 <wire x1="5" y1="25.54" x2="7.54" y2="25.54" width="0.2032" layer="16"/>
 <wire x1="7.54" y1="25.54" x2="8" y2="26" width="0.2032" layer="16"/>
-<contactref element="R8" pad="1"/>
-<wire x1="10" y1="23.95" x2="9.41" y2="24.54" width="0.508" layer="1"/>
-<wire x1="9.41" y1="24.54" x2="6" y2="24.54" width="0.508" layer="1"/>
-<wire x1="6" y1="24.54" x2="5" y2="25.54" width="0.508" layer="1"/>
-</signal>
-<signal name="N$5">
-<contactref element="K1" pad="12"/>
+</signal>
+<signal name="LED_PWM">
+<contactref element="GPIO" pad="12"/>
 <contactref element="U2" pad="2"/>
 <wire x1="7" y1="42" x2="7" y2="40.3001" width="0.2032" layer="1"/>
@@
 <contactref element="R2" pad="1"/>
 <contactref element="U1" pad="6"/>
-<contactref element="K1" pad="27"/>
+<contactref element="GPIO" pad="27"/>
 <wire x1="59" y1="39.95" x2="59" y2="44" width="0.2032" layer="1"/>
 <wire x1="59" y1="44" x2="59.365" y2="44.365" width="0.2032" layer="1"/>
@@
 <wire x1="7" y1="37.6999" x2="7" y2="36" width="0.508" layer="1"/>
 </signal>
-<signal name="N$8">
+<signal name="LED_FB">
 <contactref element="U2" pad="6"/>
 <contactref element="R4" pad="1"/>
@@
 <wire x1="13" y1="36" x2="9" y2="36" width="0.508" layer="1"/>
 </signal>
-<signal name="N$9">
+<signal name="LED_SW">
 <contactref element="U2" pad="3"/>
 <contactref element="D1" pad="A"/>
@@
 </signal>
 <signal name="LED4">
-<contactref element="K1" pad="13"/>
+<contactref element="GPIO" pad="13"/>
 <contactref element="R6" pad="1"/>
 <wire x1="14.95" y1="6" x2="14.95" y2="6.95" width="0.3048" layer="1"/>
@@
 </signal>
 <signal name="LED3">
-<contactref element="K1" pad="11"/>
+<contactref element="GPIO" pad="11"/>
 <contactref element="R5" pad="1"/>
 <wire x1="10.95" y1="6" x2="10.95" y2="6.95" width="0.3048" layer="1"/>
@@
 </signal>
 <signal name="LED5">
-<contactref element="K1" pad="15"/>
+<contactref element="GPIO" pad="15"/>
 <contactref element="R7" pad="1"/>
 <wire x1="18.95" y1="6" x2="18.95" y2="6.95" width="0.3048" layer="1"/>

Commit message: final layout?
Parts:
- R3: value 1k -> 3k9
- R4: value 0.57 -> 0.56
Connections:
- net LED_PWM renamed LED_CTRL
Changed lines of the file:
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@@
 <attribute name="VALUE" x="55.5456" y="39.285" size="2.0828" layer="27" ratio="10" rot="SR0"/>
 </element>
-<element name="R3" library="resistor" package="M0805" value="1k" x="57" y="39" smashed="yes" rot="R90">
+<element name="R3" library="resistor" package="M0805" value="3k9" x="57" y="39" smashed="yes" rot="R90">
 <attribute name="NAME" x="57" y="37" size="0.8128" layer="25" rot="R180" align="center"/>
 <attribute name="TOLERANCE" value="5%" x="57" y="39" size="1.778" layer="27" rot="R90" display="off"/>
@@
 <attribute name="VALUE" x="8.1" y="40" size="1.016" layer="27" rot="R270"/>
 </element>
-<element name="R4" library="resistor" package="M0805" value="0.57" x="9" y="33" smashed="yes" rot="R270">
+<element name="R4" library="resistor" package="M0805" value="0.56" x="9" y="33" smashed="yes" rot="R270">
 <attribute name="NAME" x="10.016" y="34.016" size="0.8128" layer="25" rot="R270"/>
 <attribute name="TOLERANCE" value="5%" x="9" y="33" size="1.778" layer="27" rot="R270" display="off"/>
@@
 <wire x1="7.54" y1="25.54" x2="8" y2="26" width="0.2032" layer="16"/>
 </signal>
-<signal name="LED_PWM">
-<contactref element="GPIO" pad="12"/>
-<contactref element="U2" pad="2"/>
-<wire x1="7" y1="42" x2="7" y2="40.3001" width="0.2032" layer="1"/>
-<via x="7" y="42" extent="1-16" drill="0.35"/>
-<wire x1="7" y1="42" x2="7" y2="48" width="0.2032" layer="16"/>
-<wire x1="7" y1="48" x2="8.3556" y2="49.3556" width="0.2032" layer="16"/>
-<wire x1="21.07" y1="53.16974375" x2="21.07" y2="53.77" width="0.2032" layer="16"/>
-<wire x1="19.6984" y1="51.79814375" x2="21.07" y2="53.16974375" width="0.2032" layer="16"/>
-<wire x1="18.09244375" y1="49.3556" x2="19.6984" y2="50.96155625" width="0.2032" layer="16"/>
-<wire x1="19.6984" y1="50.96155625" x2="19.6984" y2="51.79814375" width="0.2032" layer="16"/>
-<wire x1="8.3556" y1="49.3556" x2="18.09244375" y2="49.3556" width="0.2032" layer="16"/>
-</signal>
 <signal name="EEPROM_WP">
 <contactref element="U1" pad="7"/>
@@
 <wire x1="26.15" y1="47.15" x2="26.15" y2="51.23" width="0.3048" layer="16"/>
 </signal>
+<signal name="LED_CTRL">
+<contactref element="GPIO" pad="12"/>
+<wire x1="21.07" y1="53.77" x2="19.546" y2="52.246" width="0.2032" layer="16"/>
+<wire x1="19.546" y1="52.246" x2="19.546" y2="50.80915625" width="0.2032" layer="16"/>
+<wire x1="19.546" y1="50.80915625" x2="18.09244375" y2="49.3556" width="0.2032" layer="16"/>
+<wire x1="8.8527" y1="49.3556" x2="7" y2="47.5029" width="0.2032" layer="16"/>
+<wire x1="18.09244375" y1="49.3556" x2="8.8527" y2="49.3556" width="0.2032" layer="16"/>
+<wire x1="7" y1="47.5029" x2="7" y2="42" width="0.2032" layer="16"/>
+<contactref element="U2" pad="2"/>
+<wire x1="7" y1="40.3001" x2="7" y2="42" width="0.2032" layer="1"/>
+<via x="7" y="42" extent="1-16" drill="0.35"/>
+</signal>
 </signals>

Commit message: address drc complaints, fixed font
Parts:
- LED3: value (none) -> RED
- LED4: value (none) -> GREEN
- LED5: value (none) -> BLUE
