File: hardware/hat/scanner.brd (EAGLE design)
At the start: 65 x 56 mm, 30 parts, among them J1 PJ-102AH, U1 CAT24C32WI-GT3, U2 TPS61165DBV

Commit message: update layout
Routing:
- net LED_CTRL: track 27.6 -> 29.7 mm
- net LED_FB: track 62.5 -> 63.0 mm
Changed lines of the file:
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@@
 <wire x1="-18.8" y1="-12.55" x2="-18.8" y2="-11" width="0.508" layer="1"/>
 <via x="-18.8" y="-11" extent="1-16" drill="0.35"/>
-<wire x1="-18.8" y1="-11" x2="-18.8" y2="-3.7" width="0.508" layer="16"/>
-<wire x1="-18.8" y1="-3.7" x2="-19" y2="-3.5" width="0.508" layer="16"/>
-<wire x1="-19" y1="-3.5" x2="-19.5" y2="-3" width="0.508" layer="16"/>
-<wire x1="-19.5" y1="-3" x2="-23.5" y2="-3" width="0.508" layer="16"/>
-<wire x1="-23.5" y1="-3" x2="-24.13" y2="-2.37" width="0.508" layer="16"/>
+<wire x1="-24.13" y1="-2.37" x2="-23.5" y2="-3" width="0.508" layer="16"/>
 <wire x1="-24.13" y1="-2.37" x2="-24.13" y2="-1.27" width="0.508" layer="16"/>
 <wire x1="-3.75" y1="-2.75" x2="-4" y2="-3" width="0.508" layer="1"/>
-<wire x1="-4" y1="-3" x2="-18.5" y2="-3" width="0.508" layer="1"/>
-<wire x1="-18.5" y1="-3" x2="-19" y2="-3.5" width="0.508" layer="1"/>
-<via x="-19" y="-3.5" extent="1-16" drill="0.35"/>
+<wire x1="-18.8" y1="-3" x2="-18.8" y2="-11" width="0.508" layer="16"/>
+<via x="-18.8" y="-3" extent="1-16" drill="0.35"/>
+<wire x1="-4" y1="-3" x2="-18.8" y2="-3" width="0.508" layer="1"/>
+<wire x1="-23.5" y1="-3" x2="-18.8" y2="-3" width="0.508" layer="16"/>
 </signal>
 <signal name="EEPROM_SCL">
@@
 <wire x1="-15.0876" y1="-0.80706875" x2="-15.0876" y2="-3.15075" width="0.3048" layer="16"/>
 <wire x1="-15.532" y1="-15" x2="-16.032" y2="-15.5" width="0.3048" layer="16"/>
-<wire x1="-16.032" y1="-15.5" x2="-18.8" y2="-15.5" width="0.3048" layer="16"/>
-<via x="-18.8" y="-15.5" extent="1-16" drill="0.35"/>
-<wire x1="-18.8" y1="-15.5" x2="-18.8" y2="-14.45" width="0.3048" layer="1"/>
 <wire x1="-18.8" y1="-14.45" x2="-20.9" y2="-14.45" width="0.3048" layer="1"/>
 <wire x1="-18.8" y1="-14.45" x2="-16.7" y2="-14.45" width="0.3048" layer="1"/>
+<wire x1="-16.032" y1="-15.5" x2="-20.9" y2="-15.5" width="0.3048" layer="16"/>
+<via x="-20.9" y="-15.5" extent="1-16" drill="0.35"/>
+<wire x1="-20.9" y1="-15.5" x2="-20.9" y2="-14.45" width="0.3048" layer="1"/>
 </signal>
 <signal name="LED_COMP">
@@
 <wire x1="-24.96" y1="-17.0225" x2="-25.05" y2="-16.9325" width="0.6096" layer="1"/>
 <wire x1="-25.05" y1="-16.9325" x2="-25.05" y2="-14.8001" width="0.6096" layer="1"/>
-<wire x1="-24.96" y1="-17.0225" x2="-23.4775" y2="-17.0225" width="0.6096" layer="1"/>
-<wire x1="-22.5" y1="-18" x2="-22.5" y2="-19.5" width="0.6096" layer="1"/>
-<wire x1="-23.4775" y1="-17.0225" x2="-22.5" y2="-18" width="0.6096" layer="1"/>
-<wire x1="-22.5" y1="-19.5" x2="-21.5" y2="-20.5" width="0.6096" layer="1"/>
-<wire x1="-21.5" y1="-20.5" x2="-18.86841875" y2="-20.5" width="0.6096" layer="1"/>
-<wire x1="-18.86841875" y1="-20.5" x2="-18.86041875" y2="-20.492" width="0.6096" layer="1"/>
-<wire x1="-18.86041875" y1="-20.492" x2="-16.13958125" y2="-20.492" width="0.6096" layer="1"/>
-<wire x1="-16.13958125" y1="-20.492" x2="-16.13158125" y2="-20.5" width="0.6096" layer="1"/>
-<wire x1="18.86041875" y1="-20.492" x2="16.13958125" y2="-20.492" width="0.6096" layer="1"/>
-<wire x1="16.13158125" y1="-20.5" x2="16.13958125" y2="-20.492" width="0.6096" layer="1"/>
-<wire x1="-16.13158125" y1="-20.5" x2="16.13158125" y2="-20.5" width="0.6096" layer="1"/>
-<wire x1="20.008" y1="-31.192" x2="20.008" y2="-21.63958125" width="0.6096" layer="1"/>
-<wire x1="20.008" y1="-31.192" x2="19" y2="-32.2" width="0.6096" layer="1"/>
+<wire x1="-23.4775" y1="-17.0225" x2="-24.96" y2="-17.0225" width="0.6096" layer="1"/>
+<wire x1="21.008" y1="-30.192" x2="21.008" y2="-21.63958125" width="0.6096" layer="1"/>
+<wire x1="21.008" y1="-30.192" x2="19" y2="-32.2" width="0.6096" layer="1"/>
 <wire x1="17.5" y1="-32.2" x2="19" y2="-32.2" width="0.6096" layer="1"/>
-<wire x1="20.008" y1="-21.63958125" x2="18.86041875" y2="-20.492" width="0.6096" layer="1"/>
+<wire x1="21.008" y1="-21.63958125" x2="19.36041875" y2="-19.992" width="0.6096" layer="1"/>
+<wire x1="19.36041875" y1="-19.992" x2="-20.508" y2="-19.992" width="0.6096" layer="1"/>
+<wire x1="-20.508" y1="-19.992" x2="-23.4775" y2="-17.0225" width="0.6096" layer="1"/>
 </signal>
 <signal name="LED_SW">

Commit message: tweak layout
Parts:
- moved R10 0.10 mm to (23.9, -14.0)
Changed lines of the file:
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@@
 <attribute name="VALUE" x="29.4544" y="-3.285" size="2.0828" layer="27" ratio="10" rot="SR180"/>
 </element>
-<element name="R10" library="resistor" package="M0805" value="3k9" x="23.8" y="-14" smashed="yes" rot="R90">
-<attribute name="NAME" x="23.784" y="-16.516" size="0.8128" layer="25" font="fixed" rot="R180" align="center"/>
-<attribute name="TOLERANCE" value="5%" x="26.0225" y="-35.59" size="1.778" layer="27" rot="R90" display="off"/>
-<attribute name="VALUE" x="26.086" y="-15.016" size="1.27" layer="27" rot="R90"/>
+<element name="R10" library="resistor" package="M0805" value="3k9" x="23.9" y="-14" smashed="yes" rot="R90">
+<attribute name="NAME" x="23.884" y="-16.516" size="0.8128" layer="25" font="fixed" rot="R180" align="center"/>
+<attribute name="TOLERANCE" value="5%" x="26.1225" y="-35.59" size="1.778" layer="27" rot="R90" display="off"/>
+<attribute name="VALUE" x="26.186" y="-15.016" size="1.27" layer="27" rot="R90"/>
 </element>
 <element name="JP1" library="pinhead" library_urn="urn:adsk.eagle:library:325" package="1X02" package3d_urn="urn:adsk.eagle:package:22435/2" value="" x="26" y="-19" smashed="yes">
@@
 <contactref element="R10" pad="1"/>
 <wire x1="28.1" y1="-14.95" x2="26" y2="-14.95" width="0.508" layer="1"/>
-<wire x1="26" y1="-14.95" x2="23.8" y2="-14.95" width="0.508" layer="1"/>
-<wire x1="23.8" y1="-14.95" x2="21.45" y2="-14.95" width="0.508" layer="1"/>
+<wire x1="26" y1="-14.95" x2="23.9" y2="-14.95" width="0.508" layer="1"/>
+<wire x1="23.9" y1="-14.95" x2="21.45" y2="-14.95" width="0.508" layer="1"/>
 <wire x1="21.45" y1="-14.95" x2="21" y2="-14.5" width="0.508" layer="1"/>
 <wire x1="21" y1="-5" x2="21" y2="-11" width="0.508" layer="1"/>
@@
 <wire x1="-21.59" y1="1.27" x2="-24.13" y2="1.27" width="0.6096" layer="1"/>
 <wire x1="-20.32" y1="0" x2="-21.59" y2="1.27" width="0.6096" layer="1"/>
-<wire x1="-19.3" y1="-5.2" x2="-20.32" y2="-4.18" width="0.6096" layer="1"/>
-<wire x1="-20.32" y1="-4.18" x2="-20.32" y2="0" width="0.6096" layer="1"/>
+<wire x1="-19.2114" y1="-5.1886" x2="-20.32" y2="-4.08" width="0.6096" layer="1"/>
+<wire x1="-20.32" y1="-4.08" x2="-20.32" y2="0" width="0.6096" layer="1"/>
 <contactref element="U3" pad="3"/>
-<wire x1="-14.9012" y1="-5.1886" x2="-19.2886" y2="-5.1886" width="0.6096" layer="1"/>
-<wire x1="-19.2886" y1="-5.1886" x2="-19.3" y2="-5.2" width="0.6096" layer="1"/>
+<wire x1="-14.9012" y1="-5.1886" x2="-19.2114" y2="-5.1886" width="0.6096" layer="1"/>
 <contactref element="C6" pad="+"/>
 <contactref element="J1" pad="1"/>
@@
 <contactref element="JP1" pad="1"/>
 <contactref element="R10" pad="2"/>
-<wire x1="23.8" y1="-13.05" x2="23.8" y2="-12.7" width="0.3048" layer="1"/>
-<wire x1="25" y1="-11.5" x2="23.8" y2="-12.7" width="0.3048" layer="1"/>
+<wire x1="23.9" y1="-13.05" x2="23.9" y2="-12.6" width="0.3048" layer="1"/>
+<wire x1="25" y1="-11.5" x2="23.9" y2="-12.6" width="0.3048" layer="1"/>
 <wire x1="23.5362" y1="-9.635" x2="24.635" y2="-9.635" width="0.3048" layer="1"/>
 <wire x1="24.635" y1="-9.635" x2="25" y2="-10" width="0.3048" layer="1"/>

Commit message: v.1.1-final
Parts:
- moved C1 61.7 mm to (9.60, 39.0)
- moved C2 61.7 mm to (5.50, 34.5)
- moved C3 61.7 mm to (6.50, 30.5)
- moved C4 61.7 mm to (58.5, 47.5)
- moved C6 61.7 mm to (12.5, 13.3)
- moved D1 61.7 mm to (3.50, 34.5)
- moved GPIO 61.7 mm to (32.5, 52.5)
- moved J1 61.7 mm to (5.00, 9.00)
- moved JP1 61.7 mm to (58.5, 33.5)
- moved L1 61.7 mm to (6.50, 45.0)
- moved LED1 61.7 mm to (15.0, 25.5)
- moved LED2 61.7 mm to (50.0, 25.5)
- moved LED3 61.7 mm to (10.0, 3.00)
- moved LED4 61.7 mm to (14.0, 3.00)
- moved LED5 61.7 mm to (18.0, 3.00)
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Routing:
- net LED_FB: track 63.0 -> 64.2 mm
